Commit message: updating urdf to fix idol gear

File: rbx1_urdf/urdf/rbx1.urdf (robot description, URDF)
Before this commit: robot rbx1_urdf, 15 links, 14 joints
Links:
- removed link world
Joints:
- removed joint fixed
- joint gripper_idol_gear_joint: axis 0 1 0 -> 0 -1 0; origin xyz=-0.024233 -0.013715 -0.00052 rpy=4.71239 0.0 1.5708 -> xyz=-0.024233 -0.013715 -0.00052 rpy=1.5708 0.0 1.5708
- joint tip_gripper_idol_joint: mimic joint=gripper_idol_gear_joint multiplier=-1 offset=0 -> joint=gripper_idol_gear_joint multiplier=1 offset=0; origin xyz=-0.040206 0 -0.001701 rpy=0.0 -0.5236 -3.1416 -> xyz=-0.040206 0 -0.001701 rpy=-3.1416 0.5236 -3.1416

Commit message: Fixed endeffector coordination

File: rbx1_urdf/urdf/rbx1.urdf (robot description, URDF)
Before this commit: robot rbx1_urdf, 14 links, 13 joints
Joints:
- joint gripper_idol_gear_joint: mimic (none) -> joint=gripper_servo_gear_joint multiplier=1 offset=0
- joint joint_6_wrist_hand: limit lower=-3.141595 upper=3.141595 effort=5 velocity=1 -> (none); type revolute -> fixed
- joint pivot_arm_gripper_idol_joint: type revolute -> continuous
- joint pivot_arm_gripper_servo_joint: type revolute -> continuous
- joint tip_gripper_idol_joint: type revolute -> continuous
- joint tip_gripper_servo_joint: type revolute -> continuous
